File: design/qrng/RotationGate.kicad_sch (KiCad schematic)
At the start: 20 parts, among them Q34 NMOS, Q9 PMOS

Commit message: Updated KiCAD design
Parts:
- removed Q34: NMOS, symbol Simulation_SPICE:NMOS
- removed Q9: PMOS, symbol Simulation_SPICE:PMOS
- removed R17: 1k, symbol Device:R_Small_US
Connections:
- net SRLatch/Q renamed DFlipFlop/Out
- net SRLatch1/Q renamed DFlipFlop1/Out
- net SRLatch2/Q renamed DFlipFlop2/Out
- net SRLatch3/Q renamed DFlipFlop3/Out
- net SRLatch4/Q renamed DFlipFlop4/Out
- net SRLatch5/Q renamed DFlipFlop5/Out
- net SRLatch6/Q renamed DFlipFlop6/Out
- net SRLatch7/Q renamed DFlipFlop7/Out
- no-connect marks 10 -> 2
Other:
- removed sheet SRLatch
- removed sheet SRLatch1
- removed sheet SRLatch2
- removed sheet SRLatch3
- removed sheet SRLatch4
- removed sheet SRLatch5
- removed sheet SRLatch6
- removed sheet SRLatch7
- added sheet DFlipFlop (DFlipFlop.kicad_sch)
- added sheet DFlipFlop1 (DFlipFlop.kicad_sch)
- added sheet DFlipFlop2 (DFlipFlop.kicad_sch)
- added sheet DFlipFlop3 (DFlipFlop.kicad_sch)
- added sheet DFlipFlop4 (DFlipFlop.kicad_sch)
- added sheet DFlipFlop5 (DFlipFlop.kicad_sch)
- added sheet DFlipFlop6 (DFlipFlop.kicad_sch)
- added sheet DFlipFlop7 (DFlipFlop.kicad_sch)
- moved on the sheet: Y1
