File: design/qrng/SRLatch.kicad_sch (KiCad schematic)
At the start: 4 parts, among them Q10 NMOS, Q11 NMOS, Q12 NMOS, Q13 NMOS

Commit message: Updated KiCAD design
Parts:
- renumbered Q12 to Q11, Q11 to Q12
