File: design/qrng/UnitaryGates.kicad_sch (KiCad schematic)
At the start: 6 parts, among them M1 Measure

Commit message: Updated KiCAD design
Connections:
- net Trigger: now reaches PS1. (gnd)
- net at H1. (VOut): now also M1. (gnd); no longer PZ1. (gnd)
- net Out: now reaches M1. (gnd)
- new net: M1. (gnd), PS1. (gnd), PX1. (gnd), PY1. (gnd), PZ1. (gnd) (x2)
- new net: PS1. (gnd), PX1. (gnd)
- new net: H1. (VOut), PZ1. (gnd)
- new net: PY1. (gnd), PZ1. (gnd)
- new net: H1. (VOut), M1. (gnd)
- new net: PX1. (gnd), PY1. (gnd)
- new net D0: PX1. (gnd), PY1. (gnd), PZ1. (gnd)
- new net D1: PX1. (gnd), PY1. (gnd), PZ1. (gnd)
- new net D2: PX1. (gnd), PY1. (gnd), PZ1. (gnd)
- new net D3: PX1. (gnd), PY1. (gnd), PZ1. (gnd)
- new net D4: PX1. (gnd), PY1. (gnd), PZ1. (gnd)
- new net D5: PX1. (gnd), PY1. (gnd), PZ1. (gnd)
- new net D6: PX1. (gnd), PY1. (gnd), PZ1. (gnd)
- new net D7: PX1. (gnd), PY1. (gnd), PZ1. (gnd)
