File: design/qrng/qrng.kicad_sch (KiCad schematic)
At the start: 4 parts

Commit message: Initial commit
Parts:
- added D4, D5, D6: 1N4001, Diode_THT:D_DO-41_SOD81_P10.16mm_Horizontal, symbol Diode:1N4001
Connections:
- net at BS1.: now also D3.
- net VCC: now reaches D2.2 (A)
- net VCC: now also D1.2 (A)
- new net IN1: D5.2 (A)
- new net IN2: D4.2 (A)
- new net IN3: D6.2 (A)
- new net OUT: D4.1 (K), D5.1 (K), D6.1 (K)
Other:
- added sheet UnitaryGates (UnitaryGates.kicad_sch)
- note added: "3:1 MUX"
- note added: "Data In"
- note added: "Data Out"
- moved on the sheet: BS1, D1, D2, D3

Commit message: Updated KiCAD design
Parts:
- removed BS1: ~, symbol photonic_structures:BeamSplitter
- removed D1, D2: ~, symbol photonic_structures:PhotoDiode
- removed D3: ~, symbol photonic_structures:LED
- removed D4, D5, D6: 1N4001, Diode_THT:D_DO-41_SOD81_P10.16mm_Horizontal, symbol Diode:1N4001
- added Q153: PMOS, symbol Simulation_SPICE:PMOS
Other:
- added sheet Demux (Demux.kicad_sch)
- sheet UnitaryGates ports: added D0, D1, D2, D3, D4, D5, D6, D7, Out, Trigger, X_En, Y_En, Z_En; removed none
- note removed: "3:1 MUX"
